File: board/picopico/picopico.kicad_sch (KiCad schematic)
At the start: 52 parts, among them J2 display, J3 USB_B_Micro, Q1 BC817, Q2 BC817, SW1 SW_SPDT, SW3 SW_Push, SW5 SW_Push, SW6 SW_Push, SW7 SW_Push, SW8 SW_Push, U1 ESP32-WROVER-E, U2 volume_wheel, U3 AMS1117-3.3, U4 audio, U5 STC4054GR, U6 CH340C

Commit message: more board changes
Parts:
- added TP11, TP12: TestPoint, picopico:pad, symbol Connector:TestPoint
- BT1: footprint Connector_JST:JST_PH_S2B-PH-K_1x02_P2.00mm_Horizontal -> picopico:SM02B-SRSS-TB
- SW7, SW8: footprint Button_Switch_SMD:SW_SPST_B3U-1000P -> Button_Switch_SMD:SW_SPST_B3U-1100P-B
Connections:
- net +BATT: now also TP12.1
- net GND: now also TP11.1
Other:
- moved on the sheet: BT1, C1, C2, C3, C4, C5, J3, Q1, Q2, R1, R10, R11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

Commit message: more board stuff
Connections:
- net DTS: now reaches Q2.2 (E), R12.1, U6.13 (~{DTR})
- net RTS: now reaches Q1.2 (E), R11.1, U6.14 (~{RTS})
Other:
- note added: "5V -> 3v3"
- note added: "Audio"
- note added: "Auto program"
- note added: "Battery & Charging"
- note added: "Buttons"
- note added: "Display"
- note added: "USB IN"
- note added: "USB UART"
- moved on the sheet: C1, C2, C3, C4, J2, J3, LS1, Q1, Q2, R11, R12, R9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

Commit message: blah
Parts:
- removed U3: AMS1117-3.3, Package_TO_SOT_SMD:SOT-223-3_TabPin2, symbol Regulator_Linear:AMS1117-3.3
- added R13, R14, R15, R16, R17: 0, Resistor_SMD:R_0201_0603Metric, symbol Device:R
- added U3: AP7333-33SAG, Package_TO_SOT_SMD:SOT-23, symbol picopico:AP7333-33SAG
- J2: footprint picopico:1.77 display -> picopico:lcd smd; symbol Connector_Generic:Conn_01x08 -> Connector_Generic:Conn_01x14
Connections:
- net +3.3V: now also J2.10 (Pin_10), J2.11 (Pin_11), J2.4 (Pin_4), U3.2 (OUT); no longer J2.2 (Pin_2)
- net CS: now also R17.1; no longer J2.7 (Pin_7)
- net DC/RS: now also U1.37 (GPIO23), R14.1; no longer J2.6 (Pin_6), U1.33 (GPIO21)
- net GND: now also J2.13 (Pin_13), J2.2 (Pin_2), J2.3 (Pin_3), J2.5 (Pin_5), U3.2 (OUT); no longer J2.1 (Pin_1)
- net RESET: now also U1.16 (MTCK/GPIO13/ADC2_CH4), R13.1; no longer J2.5 (Pin_5), U1.36 (GPIO22)
- net SCK: now also U1.33 (GPIO21), R16.1; no longer J2.3 (Pin_3), U1.16 (MTCK/GPIO13/ADC2_CH4)
- net SDA: now also U1.36 (GPIO22), R15.1; no longer J2.4 (Pin_4), U1.37 (GPIO23)
- net VIN: now also U3.1 (IN)
- net LED/BL: no longer names the net of U1.30 (GPIO18)
- net LED/BL: no longer J2.8 (Pin_8)
- new net: J2.9 (Pin_9), R16.2
- new net: J2.6 (Pin_6), R13.2
- new net: J2.12 (Pin_12), R17.2
- new net: J2.7 (Pin_7), R14.2
- new net: J2.8 (Pin_8), R15.2
- no-connect marks 10 -> 15

Commit message: more boardstuff
Parts:
- removed TP1, TP2, TP3, TP4: TestPoint, picopico:pad, symbol Connector:TestPoint
- added C6: 0.1uF, Capacitor_SMD:C_1206_3216Metric, symbol Device:C
- added J1: Conn_01x04, Connector_PinHeader_2.54mm:PinHeader_1x04_P2.54mm_Vertical_SMD_Pin1Right, symbol Connector_Generic:Conn_01x04
Connections:
- net +3.3V: now also C6.1, J1.1 (Pin_1)
- net GND: now also C6.2, J1.4 (Pin_4)
- net RX: now also J1.3 (Pin_3)
- net SW_A: now also U1.29 (GPIO5); no longer U1.24 (ADC2_CH2/GPIO2)
- net SW_B: now also U1.24 (ADC2_CH2/GPIO2); no longer U1.29 (GPIO5)
- net TX: now also J1.2 (Pin_2)
- no-connect marks 15 -> 19

Commit message: board stuff
Other:
- note added: "FIXME ALL FLOATING"
Changed lines of the file:
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@@
     (effects (font (size 1.27 1.27)) (justify left bottom))
+  )
+  (text "FIXME ALL FLOATING" (at 181.61 156.21 0)
+    (effects (font (size 2 2) (thickness 0.4) bold) (justify left bottom))
   )
   (label "CS" (at 64.77 78.74 180)
